Commit message: Use CAD mesh for ROS base link

File: ros2_ws/src/robot_arm_description/urdf/robot_arm.urdf.xacro (robot description, xacro)
@@ -15,7 +15,10 @@
   <link name="base_link">
     <visual>
-      <origin xyz="0 0 0.04" rpy="0 0 0"/>
+      <!-- SolidWorks exported the mesh Y-up; rotate it into ROS Z-up. -->
+      <origin xyz="0 0 0" rpy="1.5708 0 0"/>
       <geometry>
-        <cylinder radius="0.08" length="0.08"/>
+        <mesh
+          filename="package://robot_arm_description/STL/base_link.stl"
+          scale="1 1 1"/>
       </geometry>
       <material name="dark_gray"/>

Commit message: Add CAD upper-arm mesh to ROS model

File: ros2_ws/src/robot_arm_description/urdf/robot_arm.urdf.xacro (robot description, xacro)
@@ -1,6 +1,6 @@
 <?xml version="1.0"?>
 <robot xmlns:xacro="http://www.ros.org/wiki/xacro" name="robot_arm">
-  <!-- Provisional dimensions used to verify the kinematic chain in RViz. -->
-  <xacro:property name="upper_arm_length" value="0.22"/>
+  <!-- CAD-derived upper-arm joint spacing; remaining dimensions are provisional. -->
+  <xacro:property name="upper_arm_length" value="0.12"/>
   <xacro:property name="forearm_length" value="0.18"/>
   <material name="dark_gray">
@@ -27,7 +27,10 @@
   <link name="waist_link">
     <visual>
-      <origin xyz="0 0 0.03" rpy="0 0 0"/>
+      <!-- SolidWorks exported the mesh Y-up; rotate it into ROS Z-up. -->
+      <origin xyz="0 0 0" rpy="1.5708 0 0"/>
       <geometry>
-        <cylinder radius="0.055" length="0.06"/>
+        <mesh
+          filename="package://robot_arm_description/STL/waist_link.stl"
+          scale="1 1 1"/>
       </geometry>
       <material name="dark_gray"/>
@@ -43,7 +46,10 @@
   <link name="upper_arm_link">
     <visual>
-      <origin xyz="${upper_arm_length / 2} 0 0" rpy="0 0 0"/>
+      <!-- Mesh origin is the shoulder pivot; rotate its +Y span to link +X. -->
+      <origin xyz="0 0 0" rpy="0 0 -1.5708"/>
       <geometry>
-        <box size="${upper_arm_length} 0.05 0.05"/>
+        <mesh
+          filename="package://robot_arm_description/STL/upper_arm_link.stl"
+          scale="1 1 1"/>
       </geometry>
       <material name="blue"/>

Commit message: Fix upper-arm orientation in ROS model

File: ros2_ws/src/robot_arm_description/urdf/robot_arm.urdf.xacro (robot description, xacro)
@@ -46,6 +46,6 @@
   <link name="upper_arm_link">
     <visual>
-      <!-- Mesh origin is the shoulder pivot; rotate its +Y span to link +X. -->
-      <origin xyz="0 0 0" rpy="0 0 -1.5708"/>
+      <!-- SolidWorks exports this mesh Y-up; rotate +Y to ROS +Z. -->
+      <origin xyz="0 0 0" rpy="1.5708 0 0"/>
       <geometry>
         <mesh
@@ -75,5 +75,6 @@
     <parent link="upper_arm_link"/>
     <child link="forearm_link"/>
-    <origin xyz="${upper_arm_length} 0 0" rpy="0 0 0"/>
+    <!-- The upper arm now extends along its link-frame +Z axis. -->
+    <origin xyz="0 0 ${upper_arm_length}" rpy="0 0 0"/>
     <axis xyz="0 1 0"/>
     <limit lower="-2.0944" upper="2.0944" effort="10.0" velocity="1.0"/>

Commit message: Align waist mesh with CAD base

File: ros2_ws/src/robot_arm_description/urdf/robot_arm.urdf.xacro (robot description, xacro)
@@ -40,5 +40,6 @@
     <parent link="base_link"/>
     <child link="waist_link"/>
-    <origin xyz="0 0 0.08" rpy="0 0 0"/>
+    <!-- The CAD base is 56 mm tall, so place the waist directly on its top face. -->
+    <origin xyz="0 0 0.056" rpy="0 0 0"/>
     <axis xyz="0 0 1"/>
     <limit lower="-3.1416" upper="3.1416" effort="10.0" velocity="1.0"/>

Commit message: Correct waist and upper-arm mesh axes

File: ros2_ws/src/robot_arm_description/urdf/robot_arm.urdf.xacro (robot description, xacro)
@@ -27,6 +27,6 @@
   <link name="waist_link">
     <visual>
-      <!-- SolidWorks exported the mesh Y-up; rotate it into ROS Z-up. -->
-      <origin xyz="0 0 0" rpy="1.5708 0 0"/>
+      <!-- Rotate the Y-up CAD mesh into ROS Z-up, then yaw it into the CAD assembly orientation. -->
+      <origin xyz="0 0 0" rpy="1.5708 0 1.5708"/>
       <geometry>
         <mesh
@@ -47,6 +47,6 @@
   <link name="upper_arm_link">
     <visual>
-      <!-- SolidWorks exports this mesh Y-up; rotate +Y to ROS +Z. -->
-      <origin xyz="0 0 0" rpy="1.5708 0 0"/>
+      <!-- Rotate the CAD link so its long axis follows the ROS link-frame +X axis. -->
+      <origin xyz="0 0 0" rpy="0 0 -1.5708"/>
       <geometry>
         <mesh
@@ -76,6 +76,6 @@
     <parent link="upper_arm_link"/>
     <child link="forearm_link"/>
-    <!-- The upper arm now extends along its link-frame +Z axis. -->
-    <origin xyz="0 0 ${upper_arm_length}" rpy="0 0 0"/>
+    <!-- The upper arm extends along its link-frame +X axis. -->
+    <origin xyz="${upper_arm_length} 0 0" rpy="0 0 0"/>
     <axis xyz="0 1 0"/>
     <limit lower="-2.0944" upper="2.0944" effort="10.0" velocity="1.0"/>

Commit message: Add STEP-aligned forearm ROS mesh

File: ros2_ws/src/robot_arm_description/urdf/robot_arm.urdf.xacro (robot description, xacro)
@@ -47,6 +47,9 @@
   <link name="upper_arm_link">
     <visual>
-      <!-- Rotate the CAD link so its long axis follows the ROS link-frame +X axis. -->
-      <origin xyz="0 0 0" rpy="0 0 -1.5708"/>
+      <!--
+        STEP-derived mesh transform about the shoulder-servo shaft. The STL origin
+        is 120 mm from the shoulder pivot and 10.5 mm from the link center plane.
+      -->
+      <origin xyz="0.12 -0.0105 0" rpy="-1.5708 1.5708 0"/>
       <geometry>
         <mesh
@@ -60,5 +63,6 @@
     <parent link="waist_link"/>
     <child link="upper_arm_link"/>
-    <origin xyz="0 0 0.06" rpy="0 0 0"/>
+    <!-- Shoulder-servo shaft measured from RobotArmAssembly (1).STEP. -->
+    <origin xyz="-0.01391 -0.0065 0.04028" rpy="3.1416 -1.503064 3.1416"/>
     <axis xyz="0 1 0"/>
     <limit lower="-1.5708" upper="1.5708" effort="10.0" velocity="1.0"/>
@@ -66,7 +70,14 @@
   <link name="forearm_link">
     <visual>
-      <origin xyz="${forearm_length / 2} 0 0" rpy="0 0 0"/>
+      <!--
+        STEP-derived transform relative to the corrected upper-arm mesh.
+        This SolidWorks STL is millimeter-scaled, so convert it to meters.
+      -->
+      <origin xyz="0.011847 0.010500 -0.032668"
+              rpy="-1.570796 1.222885 0"/>
       <geometry>
-        <box size="${forearm_length} 0.045 0.045"/>
+        <mesh
+          filename="package://robot_arm_description/STL/forearm_link.stl"
+          scale="0.001 0.001 0.001"/>
       </geometry>
       <material name="blue"/>

Commit message: Correct forearm STL origin offset

File: ros2_ws/src/robot_arm_description/urdf/robot_arm.urdf.xacro (robot description, xacro)
@@ -71,9 +71,11 @@
     <visual>
       <!--
-        STEP-derived transform relative to the corrected upper-arm mesh.
+        STEP-derived transform relative to the corrected upper-arm mesh. The
+        STL export shifted the Link #2 origin by +63, +19, +8 mm, so this
+        translation compensates for that shift after applying the CAD rotation.
         This SolidWorks STL is millimeter-scaled, so convert it to meters.
       -->
-      <origin xyz="0.011847 0.010500 -0.032668"
-              rpy="-1.570796 1.222885 0"/>
+      <origin xyz="0.008230 0.002500 0.033035"
+              rpy="-1.570796 1.222882 0"/>
       <geometry>
         <mesh

Commit message: Add complete wrist and gripper CAD assembly

File: ros2_ws/src/robot_arm_description/urdf/robot_arm.urdf.xacro (robot description, xacro)
@@ -3,5 +3,4 @@
   <!-- CAD-derived upper-arm joint spacing; remaining dimensions are provisional. -->
   <xacro:property name="upper_arm_length" value="0.12"/>
-  <xacro:property name="forearm_length" value="0.18"/>
   <material name="dark_gray">
     <color rgba="0.22 0.24 0.27 1"/>
@@ -94,17 +93,86 @@
     <limit lower="-2.0944" upper="2.0944" effort="10.0" velocity="1.0"/>
   </joint>
-  <link name="gripper_link">
-    <visual>
-      <origin xyz="0.04 0 0" rpy="0 0 0"/>
+  <link name="wrist_gripper_link">
+    <!-- Link #3, exported directly from RobotArmAssembly (1).STEP. -->
+    <visual name="wrist_link_visual">
+      <origin xyz="0.033726552 0.016000000 -0.093875834"
+              rpy="-3.141592654 0.347914624 -3.141592654"/>
       <geometry>
-        <box size="0.08 0.08 0.04"/>
+        <mesh
+          filename="package://robot_arm_description/STL/wrist_link.stl"
+          scale="0.001 0.001 0.001"/>
+      </geometry>
+      <material name="orange"/>
+    </visual>
+    <!-- Neutral-pose gripper assembly. Repeated parts are separate STEP occurrences. -->
+    <visual name="gripper_base_visual">
+      <origin xyz="0.017514213 0.029001510 -0.149778624"
+              rpy="2.126155499 0 -1.570796327"/>
+      <geometry>
+        <mesh filename="package://robot_arm_description/STL/gripper_base.stl"
+              scale="0.001 0.001 0.001"/>
+      </geometry>
+      <material name="orange"/>
+    </visual>
+    <visual name="left_gear_visual">
+      <origin xyz="0.017514213 0.012101510 -0.149778624"
+              rpy="-3.141592654 0.555359172 3.141592654"/>
+      <geometry>
+        <mesh filename="package://robot_arm_description/STL/gripper_gear.stl"
+              scale="0.001 0.001 0.001"/>
+      </geometry>
+      <material name="dark_gray"/>
+    </visual>
+    <visual name="right_gear_visual">
+      <origin xyz="0.022786699 0.039001227 -0.158275735"
+              rpy="-0.078000890 0.550424487 2.993259754"/>
+      <geometry>
+        <mesh filename="package://robot_arm_description/STL/gripper_gear.stl"
+              scale="0.001 0.001 0.001"/>
+      </geometry>
+      <material name="dark_gray"/>
+    </visual>
+    <visual name="left_connecting_link_visual">
+      <origin xyz="-0.010545365 0.020845127 -0.171897166"
+              rpy="0.006154655 0.555328648 -3.129919305"/>
+      <geometry>
+        <mesh filename="package://robot_arm_description/STL/gripper_connecting_link.stl"
+              scale="0.001 0.001 0.001"/>
+      </geometry>
+      <material name="blue"/>
+    </visual>
+    <visual name="right_connecting_link_visual">
+      <origin xyz="-0.010465544 0.032709649 -0.171847637"
+              rpy="0.068379906 -0.551572497 -0.129956425"/>
+      <geometry>
+        <mesh filename="package://robot_arm_description/STL/gripper_connecting_link.stl"
+              scale="0.001 0.001 0.001"/>
+      </geometry>
+      <material name="blue"/>
+    </visual>
+    <visual name="left_finger_visual">
+      <origin xyz="-0.017219319 0.016396447 -0.171330894"
+              rpy="-0.237694726 0.506818324 2.678644506"/>
+      <geometry>
+        <mesh filename="package://robot_arm_description/STL/gripper_finger.stl"
+              scale="0.001 0.001 0.001"/>
+      </geometry>
+      <material name="orange"/>
+    </visual>
+    <visual name="right_finger_visual">
+      <origin xyz="-0.019408061 0.038647484 -0.167393098"
+              rpy="-2.907517869 0.508382631 -2.686091663"/>
+      <geometry>
+        <mesh filename="package://robot_arm_description/STL/gripper_finger.stl"
+              scale="0.001 0.001 0.001"/>
       </geometry>
       <material name="orange"/>
     </visual>
   </link>
-  <joint name="gripper_mount_joint" type="fixed">
+  <joint name="wrist_gripper_mount_joint" type="fixed">
     <parent link="forearm_link"/>
-    <child link="gripper_link"/>
-    <origin xyz="${forearm_length} 0 0" rpy="0 0 0"/>
+    <child link="wrist_gripper_link"/>
+    <!-- Visual origins above are expressed directly in the forearm link frame. -->
+    <origin xyz="0 0 0" rpy="0 0 0"/>
   </joint>
 </robot>
