Commit message: Split wrist and gripper into moving joints
Replace the single fixed wrist_gripper_link with four links and add the
wrist and gripper controls.

Links:
  wrist_link, gripper_base_link, left_gripper_link, right_gripper_link

Joints:
  wrist_joint          revolute, axis 0 1 0
  gripper_base_joint   fixed
  gripper_joint        revolute, axis 0 0 1, the single gripper control
  right_gripper_joint  revolute, mimic of gripper_joint, multiplier +1

Joint State Publisher now exposes exactly five controls: base yaw,
shoulder, elbow, wrist, and gripper. The right gripper side is passive.

Derivations from the STEP assembly:
- The wrist frame's Y axis maps exactly onto the forearm frame's Y axis,
  so the wrist pitches in the same plane as the shoulder and elbow.
- Both gear frames share one spin axis: their local Z axes are exactly
  anti-parallel in the gripper-base frame (dot product -1.000000), the
  meshing-gear signature. Anti-parallel axes mean the same signed angle
  counter-rotates the sides in world space, so the mimic multiplier is
  +1 rather than -1.
- The STEP neutral pose is the closed gripper: 2.65 mm between
  fingertips at zero, opening to roughly 49 mm at 0.30 rad.

Known approximation: the real gripper is a geared four-bar closed loop,
which URDF cannot express. Each side is modelled as one rigid
gear/connector/finger group pivoting about its gear axis, so the
connector and finger do not articulate relative to their gear. This is a
tree-safe visual and workspace approximation, not a mechanism
simulation.

Provisional, not measured: wrist limits are +/-1.5708 rad and gripper
limits are 0 to 0.30 rad. Both are conservative values chosen from the
geometry and should be replaced with the physical mechanical stops.

Static validation confirms the split model reproduces the previous
single-link placement of all twelve visuals to within 1.04 nanometres,
which is the rounding of the previous file's nine-decimal literals
rather than a modelling error. Not verified at ROS runtime: the Mac has
no ROS 2 installation, so RViz and check_urdf must be run in the Ubuntu
VM.

Co-Authored-By: Claude Opus 5 <noreply@anthropic.com>

File: ros2_ws/src/robot_arm_description/urdf/robot_arm.urdf.xacro (robot description, xacro)
@@ -3,4 +3,11 @@
   <!-- CAD-derived upper-arm joint spacing; remaining dimensions are provisional. -->
   <xacro:property name="upper_arm_length" value="0.12"/>
+  <!--
+    Gripper travel. Zero is the STEP neutral pose, which is the closed gripper
+    (2.65 mm between fingertips). Positive rotation opens the jaws; 0.30 rad
+    gives roughly 49 mm of fingertip separation. This is a provisional
+    kinematic limit and should be replaced with the measured mechanical stop.
+  -->
+  <xacro:property name="gripper_open" value="0.30"/>
   <material name="dark_gray">
     <color rgba="0.22 0.24 0.27 1"/>
@@ -93,9 +100,14 @@
     <limit lower="-2.0944" upper="2.0944" effort="10.0" velocity="1.0"/>
   </joint>
-  <link name="wrist_gripper_link">
-    <!-- Link #3, exported directly from RobotArmAssembly (1).STEP. -->
+  <!--
+    Wrist. Link #3 is now its own moving link instead of part of a fixed
+    wrist_gripper_link. The joint frame is the STEP wrist frame expressed in the
+    forearm frame, so the mesh sits at the link origin and zero reproduces the
+    STEP neutral pose exactly. The wrist frame's Y axis maps onto the forearm
+    frame's Y axis, so the wrist pitches in the same plane as shoulder and elbow.
+  -->
+  <link name="wrist_link">
     <visual name="wrist_link_visual">
-      <origin xyz="0.033726552 0.016000000 -0.093875834"
-              rpy="-3.141592654 0.347914624 -3.141592654"/>
+      <origin xyz="0 0 0" rpy="0 0 0"/>
       <geometry>
         <mesh
@@ -105,8 +117,17 @@
       <material name="orange"/>
     </visual>
-    <!-- Neutral-pose gripper assembly. Repeated parts are separate STEP occurrences. -->
+  </link>
+  <joint name="wrist_joint" type="revolute">
+    <parent link="forearm_link"/>
+    <child link="wrist_link"/>
+    <origin xyz="0.033726552 0.016000000 -0.093875834"
+            rpy="-3.141592654 0.347914624 -3.141592654"/>
+    <axis xyz="0 1 0"/>
+    <limit lower="-1.5708" upper="1.5708" effort="10.0" velocity="1.0"/>
+  </joint>
+  <!-- Gripper base, rigidly bolted to the wrist. -->
+  <link name="gripper_base_link">
     <visual name="gripper_base_visual">
-      <origin xyz="0.017514213 0.029001510 -0.149778624"
-              rpy="2.126155499 0 -1.570796327"/>
+      <origin xyz="0 0 0" rpy="0 0 0"/>
       <geometry>
         <mesh filename="package://robot_arm_description/STL/gripper_base.stl"
@@ -115,7 +136,28 @@
       <material name="orange"/>
     </visual>
+  </link>
+  <joint name="gripper_base_joint" type="fixed">
+    <parent link="wrist_link"/>
+    <child link="gripper_base_link"/>
+    <origin xyz="0.034300380 0.013001510 0.047026012"
+            rpy="-1.363351778 0 -1.570796327"/>
+  </joint>
+  <!--
+    Gripper sides.
+    The real mechanism is a geared four-bar closed loop: each gear drives a
+    connecting link that drives a finger. URDF cannot express a closed kinematic
+    chain, so each side is approximated as ONE rigid body - gear, connecting
+    link, and finger together - pivoting about its gear axis. The connecting
+    link and finger therefore do not articulate relative to their gear; this is
+    a visual and workspace approximation, not a mechanism simulation.
+    Both gear frames share a common spin axis: the left and right local Z axes
+    are exactly anti-parallel in the gripper-base frame (dot product -1.000000),
+    which is the meshing-gear signature. Because the axes are anti-parallel,
+    driving both sides with the SAME signed angle produces true counter-rotation
+    in world space, so the mimic multiplier is +1, not -1.
+  -->
+  <link name="left_gripper_link">
     <visual name="left_gear_visual">
-      <origin xyz="0.017514213 0.012101510 -0.149778624"
-              rpy="-3.141592654 0.555359172 3.141592654"/>
+      <origin xyz="0 0 0" rpy="0 0 0"/>
       <geometry>
         <mesh filename="package://robot_arm_description/STL/gripper_gear.stl"
@@ -124,7 +166,35 @@
       <material name="dark_gray"/>
     </visual>
+    <visual name="left_connecting_link_visual">
+      <origin xyz="0.035504505 0.008743617 0.004000000"
+              rpy="-3.141592654 0 -0.009919099"/>
+      <geometry>
+        <mesh filename="package://robot_arm_description/STL/gripper_connecting_link.stl"
+              scale="0.001 0.001 0.001"/>
+      </geometry>
+      <material name="blue"/>
+    </visual>
+    <visual name="left_finger_visual">
+      <origin xyz="0.040876871 0.004294937 0"
+              rpy="-3.141592654 0 0.401119022"/>
+      <geometry>
+        <mesh filename="package://robot_arm_description/STL/gripper_finger.stl"
+              scale="0.001 0.001 0.001"/>
+      </geometry>
+      <material name="orange"/>
+    </visual>
+  </link>
+  <!-- Actuated gripper side. This is the single user-facing gripper control. -->
+  <joint name="gripper_joint" type="revolute">
+    <parent link="gripper_base_link"/>
+    <child link="left_gripper_link"/>
+    <origin xyz="0.016900000 0 0"
+            rpy="3.141592654 -1.570796327 -1.570796327"/>
+    <axis xyz="0 0 1"/>
+    <limit lower="0.0" upper="${gripper_open}" effort="5.0" velocity="1.0"/>
+  </joint>
+  <link name="right_gripper_link">
     <visual name="right_gear_visual">
-      <origin xyz="0.022786699 0.039001227 -0.158275735"
-              rpy="-0.078000890 0.550424487 2.993259754"/>
+      <origin xyz="0 0 0" rpy="0 0 0"/>
       <geometry>
         <mesh filename="package://robot_arm_description/STL/gripper_gear.stl"
@@ -133,7 +203,7 @@
       <material name="dark_gray"/>
     </visual>
-    <visual name="left_connecting_link_visual">
-      <origin xyz="-0.010545365 0.020845127 -0.171897166"
-              rpy="0.006154655 0.555328648 -3.129919305"/>
+    <visual name="right_connecting_link_visual">
+      <origin xyz="0.034336030 0.010701831 0.006000000"
+              rpy="0 0 -3.125893888"/>
       <geometry>
         <mesh filename="package://robot_arm_description/STL/gripper_connecting_link.stl"
@@ -142,16 +212,7 @@
       <material name="blue"/>
     </visual>
-    <visual name="right_connecting_link_visual">
-      <origin xyz="-0.010465544 0.032709649 -0.171847637"
-              rpy="0.068379906 -0.551572497 -0.129956425"/>
-      <geometry>
-        <mesh filename="package://robot_arm_description/STL/gripper_connecting_link.stl"
-              scale="0.001 0.001 0.001"/>
-      </geometry>
-      <material name="blue"/>
-    </visual>
-    <visual name="left_finger_visual">
-      <origin xyz="-0.017219319 0.016396447 -0.171330894"
-              rpy="-0.237694726 0.506818324 2.678644506"/>
+    <visual name="right_finger_visual">
+      <origin xyz="0.040292060 0.005472576 0.014500000"
+              rpy="-3.141592654 0 0.520722397"/>
       <geometry>
         <mesh filename="package://robot_arm_description/STL/gripper_finger.stl"
@@ -160,19 +221,17 @@
       <material name="orange"/>
     </visual>
-    <visual name="right_finger_visual">
-      <origin xyz="-0.019408061 0.038647484 -0.167393098"
-              rpy="-2.907517869 0.508382631 -2.686091663"/>
-      <geometry>
-        <mesh filename="package://robot_arm_description/STL/gripper_finger.stl"
-              scale="0.001 0.001 0.001"/>
-      </geometry>
-      <material name="orange"/>
-    </visual>
-  </link>
-  <joint name="wrist_gripper_mount_joint" type="fixed">
-    <parent link="forearm_link"/>
-    <child link="wrist_gripper_link"/>
-    <!-- Visual origins above are expressed directly in the forearm link frame. -->
-    <origin xyz="0 0 0" rpy="0 0 0"/>
+  </link>
+  <!--
+    Mirrored side. The mimic tag keeps this passive, so joint_state_publisher_gui
+    exposes exactly five controls: base yaw, shoulder, elbow, wrist, and gripper.
+  -->
+  <joint name="right_gripper_joint" type="revolute">
+    <parent link="gripper_base_link"/>
+    <child link="right_gripper_link"/>
+    <origin xyz="-0.009999717 -0.010000000 0"
+            rpy="1.570796327 -1.444499427 3.141592654"/>
+    <axis xyz="0 0 1"/>
+    <limit lower="0.0" upper="${gripper_open}" effort="5.0" velocity="1.0"/>
+    <mimic joint="gripper_joint" multiplier="1.0" offset="0.0"/>
   </joint>
 </robot>

Commit message: Add fitted collision geometry and RViz configs
Add one simplified collision primitive per physical link, fitted to the
committed meshes rather than hand-estimated.

Primitive choice is data-driven, not assumed:
- base_link uses a cylinder. The mesh is genuinely round: 40.5% of its
  vertices lie in the outer 10% of radius, and a cylinder is 21%
  tighter than the bounding box.
- waist_link uses a box. It looks round but is not - only 8% of
  vertices lie in the outer 10% of radius, so a cylinder would be just
  8% tighter and the box is simpler.
- The upper arm, forearm, wrist, and gripper base use oriented boxes
  sized to each mesh's own bounding box, inheriting the mesh
  orientation rather than inflating an axis-aligned box.
- Each gripper side gets collision on the finger only. The gears and
  connecting links mesh and overlap by design, so collision geometry
  there would create permanent contact for no benefit.

Expected overlap: the two finger boxes intersect at neutral because the
gripper is closed there. Self-collision between left_gripper_link and
right_gripper_link must be disabled downstream via Gazebo self_collide
and the MoveIt SRDF. Documented rather than worked around.

Also adds the package's own RViz configs, replacing the borrowed
urdf_launch/urdf.rviz so display settings are under version control:
- rviz/robot_arm.rviz            normal visual view
- rviz/robot_arm_collision.rviz  collision primitives with meshes at 35%
                                 alpha, for visual verification

display.launch.py gains show_collision, rviz_config, and gui arguments,
and now sets all three software-rendering variables the UTM VM needs.

The validator gains a collision section: every link has a primitive, no
link uses a mesh as collision geometry, and 100% of sampled visual
vertices fall inside the matching primitive (with the internal-mechanism
meshes asserted as deliberately uncovered). All checks pass locally.

Not verified at ROS runtime: RViz rendering of the collision config and
the new launch arguments must be exercised in the Ubuntu VM.

Co-Authored-By: Claude Opus 5 <noreply@anthropic.com>

File: ros2_ws/src/robot_arm_description/urdf/robot_arm.urdf.xacro (robot description, xacro)
@@ -30,4 +30,12 @@
       <material name="dark_gray"/>
     </visual>
+    <!-- Collision: Cylinder: the base is genuinely round (40.5% of vertices lie in the outer 10% of
+         radius) and a cylinder is 21% tighter than the bounding box. -->
+    <collision>
+      <origin xyz="0 -1.02849746e-07 0.0280000009" rpy="3.6732051e-06 -0 0"/>
+      <geometry>
+        <cylinder radius="0.0606250025" length="0.0560000017"/>
+      </geometry>
+    </collision>
   </link>
   <link name="waist_link">
@@ -42,4 +50,12 @@
       <material name="dark_gray"/>
     </visual>
+    <!-- Collision: Box: the waist is NOT round - only 8% of vertices lie in the outer 10% of radius,
+         and a cylinder would be just 8% tighter than the box. Box chosen on that evidence. -->
+    <collision>
+      <origin xyz="1.35541332e-07 4.97871113e-13 0.0369000174" rpy="1.5708 -0 1.5708"/>
+      <geometry>
+        <box size="0.0968577415 0.0738000348 0.0970000029"/>
+      </geometry>
+    </collision>
   </link>
   <joint name="base_yaw_joint" type="revolute">
@@ -65,4 +81,11 @@
       <material name="blue"/>
     </visual>
+    <!-- Collision: Box sized to the mesh bounding box in its own frame. -->
+    <collision>
+      <origin xyz="0.0599999609 -2.2053394e-07 2.2039245e-07" rpy="1.57079265 1.57079265 3.14159265"/>
+      <geometry>
+        <box size="0.0419998914 0.16196901 0.0209999997"/>
+      </geometry>
+    </collision>
   </link>
   <joint name="shoulder_joint" type="revolute">
@@ -91,4 +114,11 @@
       <material name="blue"/>
     </visual>
+    <!-- Collision: Box sized to the mesh bounding box in its own frame. -->
+    <collision>
+      <origin xyz="0.0119116915 0.0160000062 -0.0331393786" rpy="-1.570796 1.222882 0"/>
+      <geometry>
+        <box size="0.124999993 0.037999997 0.027"/>
+      </geometry>
+    </collision>
   </link>
   <joint name="elbow_joint" type="revolute">
@@ -117,4 +147,11 @@
       <material name="orange"/>
     </visual>
+    <!-- Collision: Box sized to the mesh bounding box in its own frame. -->
+    <collision>
+      <origin xyz="0 0 0.023" rpy="0 -0 0"/>
+      <geometry>
+        <box size="0.033 0.028 0.046"/>
+      </geometry>
+    </collision>
   </link>
   <joint name="wrist_joint" type="revolute">
@@ -136,4 +173,12 @@
       <material name="orange"/>
     </visual>
+    <!-- Collision: Box sized to the mesh bounding box. Loose (7.2x the true volume) because the
+         part is an open forked bracket; a convex hull would be tighter if needed. -->
+    <collision>
+      <origin xyz="0.0116501546 0.0139999983 -0.0134966087" rpy="0 -0 0"/>
+      <geometry>
+        <box size="0.0532997427 0.0279999996 0.0770036621"/>
+      </geometry>
+    </collision>
   </link>
   <joint name="gripper_base_joint" type="fixed">
@@ -184,4 +229,12 @@
       <material name="orange"/>
     </visual>
+    <!-- Collision: Finger only. The gear and connecting link are internal mechanism that mesh and
+         overlap by design, so collision geometry there would create permanent contact. -->
+    <collision>
+      <origin xyz="0.0576946969 0.00715333915 -0.00224999852" rpy="3.14159265 -0 0.401119022"/>
+      <geometry>
+        <box size="0.0651637421 0.0178700542 0.00450000009"/>
+      </geometry>
+    </collision>
   </link>
   <!-- Actuated gripper side. This is the single user-facing gripper control. -->
@@ -221,4 +274,11 @@
       <material name="orange"/>
     </visual>
+    <!-- Collision: Finger only, mirroring the left side. -->
+    <collision>
+      <origin xyz="0.0566486799 0.0103172343 0.0122500015" rpy="3.14159265 -0 0.520722397"/>
+      <geometry>
+        <box size="0.0651637421 0.0178700542 0.00450000009"/>
+      </geometry>
+    </collision>
   </link>
   <!--
